File: bhdl-test/out/onebutton/one/out.kicad_pcb (KiCad board)
At the start: 2 copper layers, 80.9 x 23.8 mm, 10 parts

Commit message: add all kicad_pcb output files
Connections:
- D4 pad 2: 3 -> 1
- LED6 pad 1: 1 -> 3
- LED6 pad 2: 1 -> 3
- R2 pad 1: 3 -> 1
- R7 pad 1: 1 -> 3
- R7 pad 2: 1 -> 3
- R8 pad 1: 1 -> 3
- R8 pad 2: 1 -> 3
- U1 pad 1: 3 -> 1
- U1 pad 2: 3 -> 1
- U10 pad 1: 1 -> 3
- U10 pad 2: 1 -> 3
- U10 pad 3: 1 -> 3
- U10 pad 8: 3 -> 1
- U5 pad 1: 1 -> 3
- U9 pad 1: 1 -> 3
- U9 pad 2: 3 -> 1
Changed lines of the file:
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@@
     (drill 1.1)
     (layers *.Cu *.Mask)
-    (net 3 "3"))
+    (net 1 "1"))
    (pad
     1
@@
     (drill 1.1)
     (layers *.Cu *.Mask)
-    (net 3 "3"))
+    (net 1 "1"))
    (pad
     2
@@
     (drill 1.1)
     (layers *.Cu *.Mask)
-    (net 3 "3"))
+    (net 1 "1"))
    (pad
     1
@@
     (drill 1.1)
     (layers *.Cu *.Mask)
-    (net 3 "3"))
+    (net 1 "1"))
    (fp_text
     user
@@
     (size 0.875 0.95)
     (layers F.Cu F.Paste F.Mask)
-    (net 3 "3"))
+    (net 1 "1"))
    (pad
     2
@@
     (drill 0.8)
     (layers *.Cu *.Mask)
-    (net 3 "3"))
+    (net 1 "1"))
    (fp_text
     user
@@
     (size 0.6999985999999999 1.2500101999999997)
     (layers F.Cu F.Paste F.Mask)
-    (net 1 "1"))
+    (net 3 "3"))
    (fp_text
     user
@@
     (drill 0.8)
     (layers *.Cu *.Mask)
-    (net 1 "1"))
+    (net 3 "3"))
    (pad
     2
@@
     (drill 0.8)
     (layers *.Cu *.Mask)
-    (net 1 "1"))
+    (net 3 "3"))
    (fp_text
     user
@@
     (size 0.875 0.95)
     (layers F.Cu F.Paste F.Mask)
-    (net 1 "1"))
+    (net 3 "3"))
    (pad
     2
@@
     (size 0.875 0.95)
     (layers F.Cu F.Paste F.Mask)
-    (net 1 "1"))
+    (net 3 "3"))
    (fp_text
     user
@@
     (size 0.875 0.95)
     (layers F.Cu F.Paste F.Mask)
-    (net 1 "1"))
+    (net 3 "3"))
    (pad
     2
@@
     (size 0.875 0.95)
     (layers F.Cu F.Paste F.Mask)
-    (net 1 "1"))
+    (net 3 "3"))
    (fp_text
     user
@@
     (drill 1.0)
     (layers *.Cu *.Mask)
-    (net 1 "1"))
+    (net 3 "3"))
    (pad
     2
@@
     (drill 1.0)
     (layers *.Cu *.Mask)
-    (net 3 "3"))
+    (net 1 "1"))
    (fp_text
     user
@@
     (size 1.7999964 1.7999964)
     (layers F.Cu F.Paste F.Mask)
-    (net 3 "3"))
+    (net 1 "1"))
    (pad
     7
@@
     (size 1.7999964 1.7999964)
     (layers F.Cu F.Paste F.Mask)
-    (net 1 "1"))
+    (net 3 "3"))
    (pad
     2
@@
     (size 1.7999964 1.7999964)
     (layers F.Cu F.Paste F.Mask)
-    (net 1 "1"))
+    (net 3 "3"))
    (pad
     1
@@
     (size 1.7999964 1.7999964)
     (layers F.Cu F.Paste F.Mask)
-    (net 1 "1"))
-   (fp_text
-    user
+    (net 3 "3"))
+   (fp_text
+    user
