File: bhdl-test/out/onebutton/three/out.kicad_pcb (KiCad board)
At the start: 2 copper layers, 104.2 x 31.8 mm, 22 parts

Commit message: add all kicad_pcb output files
Connections:
- C10 pad 1: 1 -> 5
- C10 pad 2: 1 -> 5
- C15 pad 1: 2 -> 1
- C15 pad 2: 2 -> 1
- C5 pad 1: 4 -> 3
- C5 pad 2: 4 -> 3
- D11 pad 1: 1 -> 5
- D11 pad 2: 5 -> 4
- D16 pad 1: 2 -> 1
- D16 pad 2: 5 -> 4
- D6 pad 1: 4 -> 3
- D6 pad 2: 5 -> 4
- LED13 pad 1: 3 -> 2
- LED13 pad 2: 3 -> 2
- LED18 pad 1: 3 -> 2
- LED18 pad 2: 3 -> 2
- LED8 pad 1: 3 -> 2
- LED8 pad 2: 3 -> 2
- R14 pad 1: 5 -> 4
- R14 pad 2: 2 -> 1
- R19 pad 1: 3 -> 2
- R19 pad 2: 3 -> 2
- R20 pad 1: 3 -> 2
- R20 pad 2: 3 -> 2
- R4 pad 1: 5 -> 4
- R4 pad 2: 4 -> 3
- R9 pad 1: 5 -> 4
- R9 pad 2: 1 -> 5
- U1 pad 1: 5 -> 4
- U1 pad 2: 5 -> 4
- U12 pad 1: 3 -> 2
- U12 pad 3: 1 -> 5
- U17 pad 1: 3 -> 2
- U17 pad 3: 2 -> 1
- U2 pad 1: 5 -> 4
- U2 pad 2: 5 -> 4
- U21 pad 1: 3 -> 2
- U21 pad 2: 5 -> 4
- U22 pad 1: 3 -> 2
- U22 pad 2: 3 -> 2
- U22 pad 3: 3 -> 2
- U22 pad 8: 5 -> 4
- U3 pad 1: 5 -> 4
- U3 pad 2: 5 -> 4
- U7 pad 1: 3 -> 2
- U7 pad 3: 4 -> 3
Changed lines of the file:
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@@
     (drill 1.1)
     (layers *.Cu *.Mask)
-    (net 5 "5"))
+    (net 4 "4"))
    (pad
     1
@@
     (drill 1.1)
     (layers *.Cu *.Mask)
-    (net 5 "5"))
+    (net 4 "4"))
    (pad
     2
@@
     (drill 1.1)
     (layers *.Cu *.Mask)
-    (net 5 "5"))
+    (net 4 "4"))
    (pad
     1
@@
     (drill 1.1)
     (layers *.Cu *.Mask)
-    (net 5 "5"))
+    (net 4 "4"))
    (fp_text
     user
@@
     (drill 1.1)
     (layers *.Cu *.Mask)
-    (net 5 "5"))
+    (net 4 "4"))
    (pad
     1
@@
     (drill 1.1)
     (layers *.Cu *.Mask)
-    (net 5 "5"))
+    (net 4 "4"))
    (pad
     2
@@
     (drill 1.1)
     (layers *.Cu *.Mask)
-    (net 5 "5"))
+    (net 4 "4"))
    (pad
     1
@@
     (drill 1.1)
     (layers *.Cu *.Mask)
-    (net 5 "5"))
+    (net 4 "4"))
    (fp_text
     user
@@
     (drill 1.1)
     (layers *.Cu *.Mask)
-    (net 5 "5"))
+    (net 4 "4"))
    (pad
     1
@@
     (drill 1.1)
     (layers *.Cu *.Mask)
-    (net 5 "5"))
+    (net 4 "4"))
    (pad
     2
@@
     (drill 1.1)
     (layers *.Cu *.Mask)
-    (net 5 "5"))
+    (net 4 "4"))
    (pad
     1
@@
     (drill 1.1)
     (layers *.Cu *.Mask)
-    (net 5 "5"))
+    (net 4 "4"))
    (fp_text
     user
@@
     (size 0.875 0.95)
     (layers F.Cu F.Paste F.Mask)
-    (net 5 "5"))
+    (net 4 "4"))
    (pad
     2
@@
     (size 0.875 0.95)
     (layers F.Cu F.Paste F.Mask)
-    (net 4 "4"))
+    (net 3 "3"))
    (fp_text
     user
@@
     (size 0.875 0.95)
     (layers F.Cu F.Paste F.Mask)
-    (net 4 "4"))
+    (net 3 "3"))
    (pad
     2
@@
     (size 0.875 0.95)
     (layers F.Cu F.Paste F.Mask)
-    (net 4 "4"))
+    (net 3 "3"))
    (fp_text
     user
@@
     (drill 0.8)
     (layers *.Cu *.Mask)
-    (net 4 "4"))
+    (net 3 "3"))
    (pad
     2
@@
     (drill 0.8)
     (layers *.Cu *.Mask)
-    (net 5 "5"))
+    (net 4 "4"))
    (fp_text
     user
@@
     (size 0.6999985999999999 1.2500101999999997)
     (layers F.Cu F.Paste F.Mask)
-    (net 4 "4"))
+    (net 3 "3"))
    (pad
     2
@@
     (size 0.6999985999999999 1.2500101999999997)
     (layers F.Cu F.Paste F.Mask)
-    (net 3 "3"))
+    (net 2 "2"))
    (fp_text
     user
@@
     (drill 0.8)
     (layers *.Cu *.Mask)
-    (net 3 "3"))
+    (net 2 "2"))
    (pad
     2
@@
     (drill 0.8)
     (layers *.Cu *.Mask)
-    (net 3 "3"))
+    (net 2 "2"))
    (fp_text
     user
@@
     (size 0.875 0.95)
     (layers F.Cu F.Paste F.Mask)
-    (net 5 "5"))
+    (net 4 "4"))
    (pad
     2
@@
     (size 0.875 0.95)
     (layers F.Cu F.Paste F.Mask)
-    (net 1 "1"))
+    (net 5 "5"))
    (fp_text
     user
@@
     (size 0.875 0.95)
     (layers F.Cu F.Paste F.Mask)
-    (net 1 "1"))
+    (net 5 "5"))
    (pad
     2
@@
     (size 0.875 0.95)
     (layers F.Cu F.Paste F.Mask)
-    (net 1 "1"))
+    (net 5 "5"))
    (fp_text
     user
@@
     (drill 0.8)
     (layers *.Cu *.Mask)
-    (net 1 "1"))
+    (net 5 "5"))
    (pad
     2
@@
     (drill 0.8)
     (layers *.Cu *.Mask)
-    (net 5 "5"))
+    (net 4 "4"))
    (fp_text
     user
@@
     (size 0.6999985999999999 1.2500101999999997)
     (layers F.Cu F.Paste F.Mask)
-    (net 1 "1"))
+    (net 5 "5"))
    (pad
     2
@@
     (size 0.6999985999999999 1.2500101999999997)
     (layers F.Cu F.Paste F.Mask)
-    (net 3 "3"))
+    (net 2 "2"))
    (fp_text
     user
@@
     (drill 0.8)
     (layers *.Cu *.Mask)
-    (net 3 "3"))
+    (net 2 "2"))
    (pad
     2
@@
     (drill 0.8)
     (layers *.Cu *.Mask)
-    (net 3 "3"))
+    (net 2 "2"))
    (fp_text
     user
@@
     (size 0.875 0.95)
     (layers F.Cu F.Paste F.Mask)
-    (net 5 "5"))
+    (net 4 "4"))
    (pad
     2
@@
     (size 0.875 0.95)
     (layers F.Cu F.Paste F.Mask)
-    (net 2 "2"))
+    (net 1 "1"))
    (fp_text
     user
@@
     (size 0.875 0.95)
     (layers F.Cu F.Paste F.Mask)
-    (net 2 "2"))
+    (net 1 "1"))
    (pad
     2
@@
     (size 0.875 0.95)
     (layers F.Cu F.Paste F.Mask)
-    (net 2 "2"))
+    (net 1 "1"))
    (fp_text
     user
@@
     (drill 0.8)
     (layers *.Cu *.Mask)
-    (net 2 "2"))
+    (net 1 "1"))
    (pad
     2
@@
     (drill 0.8)
     (layers *.Cu *.Mask)
-    (net 5 "5"))
+    (net 4 "4"))
    (fp_text
     user
@@
     (size 0.6999985999999999 1.2500101999999997)
     (layers F.Cu F.Paste F.Mask)
-    (net 2 "2"))
+    (net 1 "1"))
    (pad
     2
@@
     (size 0.6999985999999999 1.2500101999999997)
     (layers F.Cu F.Paste F.Mask)
-    (net 3 "3"))
+    (net 2 "2"))
    (fp_text
     user
@@
     (drill 0.8)
     (layers *.Cu *.Mask)
-    (net 3 "3"))
+    (net 2 "2"))
    (pad
     2
@@
     (drill 0.8)
     (layers *.Cu *.Mask)
-    (net 3 "3"))
+    (net 2 "2"))
    (fp_text
     user
@@
     (size 0.875 0.95)
     (layers F.Cu F.Paste F.Mask)
-    (net 3 "3"))
+    (net 2 "2"))
    (pad
     2
@@
     (size 0.875 0.95)
     (layers F.Cu F.Paste F.Mask)
-    (net 3 "3"))
+    (net 2 "2"))
    (fp_text
     user
@@
     (size 0.875 0.95)
     (layers F.Cu F.Paste F.Mask)
-    (net 3 "3"))
+    (net 2 "2"))
    (pad
     2
@@
     (size 0.875 0.95)
     (layers F.Cu F.Paste F.Mask)
-    (net 3 "3"))
+    (net 2 "2"))
    (fp_text
     user
@@
     (drill 1.0)
     (layers *.Cu *.Mask)
-    (net 3 "3"))
+    (net 2 "2"))
    (pad
     2
@@
     (drill 1.0)
     (layers *.Cu *.Mask)
-    (net 5 "5"))
+    (net 4 "4"))
    (fp_text
     user
@@
     (size 1.7999964 1.7999964)
     (layers F.Cu F.Paste F.Mask)
-    (net 5 "5"))
+    (net 4 "4"))
    (pad
     7
@@
     (size 1.7999964 1.7999964)
     (layers F.Cu F.Paste F.Mask)
-    (net 3 "3"))
+    (net 2 "2"))
    (pad
     2
@@
     (size 1.7999964 1.7999964)
     (layers F.Cu F.Paste F.Mask)
-    (net 3 "3"))
+    (net 2 "2"))
    (pad
     1
@@
     (size 1.7999964 1.7999964)
     (layers F.Cu F.Paste F.Mask)
-    (net 3 "3"))
-   (fp_text
-    user
+    (net 2 "2"))
+   (fp_text
+    user
